File: PCB/PistonPump.kicad_pcb (KiCad board)
At the start: 2 copper layers, 4 parts

Commit message: pcb
Parts:
- removed REF** (x2): PhoenixContact_MSTBA-G_10x5.08mm_Angled, Connectors_Phoenix:PhoenixContact_MSTBA-G_10x5.08mm_Angled
- removed REF** (x2): Pin_Header_Straight_1x14_Pitch2.54mm, Pin_Headers:Pin_Header_Straight_1x14_Pitch2.54mm
- added C1: CP, Capacitor_THT:CP_Radial_D8.0mm_P2.50mm, F.Cu at (171.4, 108.0)
- added C2: CP, Capacitor_THT:CP_Radial_D8.0mm_P2.50mm, F.Cu at (113.0, 107.3)
- added C3: CP, Capacitor_THT:CP_Radial_D8.0mm_P2.50mm, F.Cu at (144.1, 108.0)
- added C4: CP, Capacitor_THT:CP_Radial_D8.0mm_P2.50mm, F.Cu at (172.7, 133.3)
- added C5: CP, Capacitor_THT:CP_Radial_D8.0mm_P2.50mm, F.Cu at (147.3, 133.3)
- added C6: CP, Capacitor_THT:CP_Radial_D8.0mm_P2.50mm, F.Cu at (109.9, 133.3)
- added J1: Conn_01x06, piston_pump:MOLEX_0395021006, F.Cu at (166.4, 139.7)
- added J2: Conn_01x08, piston_pump:TE_284512-8, F.Cu at (143.5, 139.7)
- added J3: Conn_01x08, piston_pump:TE_284512-8, F.Cu at (108.6, 139.7)
- added J4: Conn_01x14_Male, Connector_PinHeader_2.54mm:PinHeader_1x14_P2.54mm_Vertical, F.Cu at (147.3, 99.1)
- added J5: Conn_01x14_Male, Connector_PinHeader_2.54mm:PinHeader_1x14_P2.54mm_Vertical, F.Cu at (147.3, 119.4)
- added R1: R_US, Resistor_THT:R_Axial_DIN0204_L3.6mm_D1.6mm_P5.08mm_Horizontal, F.Cu at (124.2, 130.4)
- added R2: R_US, Resistor_THT:R_Axial_DIN0204_L3.6mm_D1.6mm_P5.08mm_Horizontal, F.Cu at (118.7, 129.9)
- added R3: R_US, Resistor_THT:R_Axial_DIN0204_L3.6mm_D1.6mm_P5.08mm_Horizontal, F.Cu at (99.7, 134.0)
- added R4: R_US, Resistor_THT:R_Axial_DIN0204_L3.6mm_D1.6mm_P5.08mm_Horizontal, F.Cu at (96.1, 126.4)
- added U2: BOB-12009, piston_pump:CONV_BOB-12009, F.Cu at (170.2, 120.7)
- added U3: BOB-12009, piston_pump:CONV_BOB-12009, F.Cu at (146.1, 120.0)
- added U4: BOB-12009, piston_pump:CONV_BOB-12009, F.Cu at (111.8, 120.7)
Routing:
- net Net-(J5-Pad6): track 0.00 -> 43.5 mm
- net Net-(J5-Pad7): track 0.00 -> 43.5 mm
- net Net-(J4-Pad13): track 0.00 -> 31.0 mm
- net Net-(J4-Pad4): track 0.00 -> 29.8 mm
- net Net-(J4-Pad6): track 0.00 -> 25.2 mm
- net Net-(J1-Pad5): track 0.00 -> 23.0 mm
- net Net-(J4-Pad14): track 0.00 -> 22.2 mm
- net Net-(J4-Pad8): track 0.00 -> 20.7 mm
- net Net-(J3-Pad2): track 0.00 -> 19.9 mm
- net Net-(J3-Pad8): track 0.00 -> 18.9 mm
- net Net-(J3-Pad4): track 0.00 -> 16.9 mm
- net Net-(J3-Pad6): track 0.00 -> 16.9 mm
- net Net-(J2-Pad4): track 0.00 -> 16.9 mm
- net Net-(J2-Pad6): track 0.00 -> 16.5 mm
- net Net-(J2-Pad2): track 0.00 -> 14.7 mm
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- added copper zone on F.Cu, net +5V
- added copper zone on F.Cu, net +5VD
- added copper zone on F.Cu, net /3V3
- added copper zone on B.Cu, net GND
Other:
- board outline added: 94 x 59.1 mm
- board text added: "+"
- board text added: "-"
- board text added: "5V"
- board text added: "AREF"
- board text added: "D5"
- board text added: "DIR"
- board text added: "ENA"
- board text added: "ESTP"
- board text added: "FSW"
- board text added: "GND"
- board text added: "MAXSW"
- board text added: "MINSW"
- board text added: "PUL"
- board text added: "Piston Pump IO Interface by Joseffus Santos joseffus@isntos.com"
- board text added: "RX"
- board text added: "TX"
