File: PCB/PistonPump_smd/PistonPump_smd.kicad_pcb (KiCad board)
At the start: 2 copper layers, 94 x 66 mm, 57 parts, among them J1 Conn_01x14_Male, J2 Conn_01x14_Male, J3 Conn_01x06, J4 Conn_01x08, J5 Conn_01x08, Q1 BSS138, Q2 BSS138, Q3 BSS138, Q4 BSS138, Q5 BSS138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

Commit message: current
Routing:
- net LV4: track 18.5 -> 23.5 mm
- net LV1: track 55.6 -> 54.5 mm
